File: MCU.sch (EAGLE design)
At the start: 2 parts, among them U1 ATXMEGA128A4U-AU

Commit message: add another line
Connections:
- new net N$10: J1.11, U1.PB2
Changed lines of the file:
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@@
+</segment>
+</net>
+<net name="N$10" class="0">
+<segment>
+<pinref part="U1" gate="G$1" pin="PB2"/>
+<pinref part="J1" gate="G$1" pin="11"/>
+<wire x1="88.9" y1="-30.48" x2="119.38" y2="-30.48" width="0.1524" layer="91"/>
+<wire x1="119.38" y1="-30.48" x2="119.38" y2="-27.94" width="0.1524" layer="91"/>
 </segment>
 </net>
